File: esp32_pcb/esp32_doorbot.kicad_sch (KiCad schematic)
At the start: 16 parts, among them J1 Conn_01x07_Male, J2 Conn_01x02_Female, J3 Barrel_Jack, J4 WROOM32_1, J5 WROOM32_2, Q1 NDT3055, U1 L7805

Commit message: Gerber/drill files for PCBWay
Parts:
- U1: Digikey # 1470-VR10S05-ND -> 1470-3971-ND
Changed lines of the file:
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@@
 			)
 		)
-		(property "Digikey #" "1470-VR10S05-ND"
+		(property "Digikey #" "1470-3971-ND"
 			(at 74.93 96.52 0)
 			(effects
